Commit message: Added discretization

File: mouse_description/urdf/mouse.xacro (robot description, xacro)
@@ -130,240 +130,3 @@
 		</plugin>
 	</gazebo>
-	<!-- Sensors -->
-	<!-- Color Sensor (Camera) -->
-	<link name="front_cam">
-		<visual>
-			<geometry>
-				<box size="0.008 0.008 0.008"/>
-			</geometry>
-		</visual>
-		<collision name="front_cam_collision">
-			<geometry>
-				<box size="0.008 0.008 0.008"/>
-			</geometry>
-		</collision>
-		<inertial>
-			<mass value="1e-5"/>
-			<inertia
-        		ixx="1e-6" ixy="0.0" ixz="0.0"
-        		iyy="1e-6" iyz="0.0"
-        		izz="1e-6"/>
-		</inertial>
-	</link>
-	<joint name="front_cam_mnt" type="fixed">
-		<origin xyz="0 0 0.027" rpy="0 0 1.5708"/>
-		<parent link="base_link"/>
-		<child link="front_cam"/>
-	</joint>
-	<gazebo reference="front_cam">
-		<material>Gazebo/Blue</material>
-		<sensor name="front_cam" type="camera">
-			<update_rate>30</update_rate>
-			<camera name="front_cam">
-				<horizontal_fov>2</horizontal_fov>
-				<image>
-					<width>640</width>
-					<height>480</height>
-					<format>R8G8B8</format>
-				</image>
-				<clip>
-					<near>0.001</near>
-					<far>0.5</far>
-				</clip>
-			</camera>
-			<plugin name="gazebo_ros_camera" filename="libgazebo_ros_camera.so">
-				<imageTopicName>image_raw</imageTopicName>
-				<cameraInfoTopicName>camera_info</cameraInfoTopicName>
-				<!-- incorrect TF frame -->
-				<frameName>base</frameName>
-			</plugin>
-		</sensor>
-	</gazebo>
-	<!-- Bumper sensor -->
-	<link name="left_bump">
-		<visual>
-			<geometry>
-				<sphere radius="0.005"/>
-			</geometry>
-		</visual>
-		<collision name="left_bump_collision">
-			<geometry>
-				<sphere radius="0.005"/>
-			</geometry>
-		</collision>
-		<inertial>
-			<mass value="1e-5"/>
-			<inertia
-        		ixx="1e-6" ixy="0.0" ixz="0.0"
-        		iyy="1e-6" iyz="0.0"
-        		izz="1e-6"/>
-		</inertial>
-	</link>
-	<link name="right_bump">
-		<visual>
-			<geometry>
-				<sphere radius="0.005"/>
-			</geometry>
-		</visual>
-		<collision name="right_bump_collision">
-			<geometry>
-				<sphere radius="0.005"/>
-			</geometry>
-		</collision>
-		<inertial>
-			<mass value="1e-5"/>
-			<inertia
-        		ixx="1e-6" ixy="0.0" ixz="0.0"
-        		iyy="1e-6" iyz="0.0"
-        		izz="1e-6"/>
-		</inertial>
-	</link>
-	<link name="left_front_bump">
-		<visual>
-			<geometry>
-				<sphere radius="0.005"/>
-			</geometry>
-		</visual>
-		<collision name="left_front_bump_collision">
-			<geometry>
-				<sphere radius="0.005"/>
-			</geometry>
-		</collision>
-		<inertial>
-			<mass value="1e-5"/>
-			<inertia
-        		ixx="1e-6" ixy="0.0" ixz="0.0"
-        		iyy="1e-6" iyz="0.0"
-        		izz="1e-6"/>
-		</inertial>
-	</link>
-	<link name="right_front_bump">
-		<visual>
-			<geometry>
-				<sphere radius="0.005"/>
-			</geometry>
-		</visual>
-		<collision name="right_front_bump_collision">
-			<geometry>
-				<sphere radius="0.005"/>
-			</geometry>
-		</collision>
-		<inertial>
-			<mass value="1e-5"/>
-			<inertia
-        		ixx="1e-6" ixy="0.0" ixz="0.0"
-        		iyy="1e-6" iyz="0.0"
-        		izz="1e-6"/>
-		</inertial>
-	</link>
-	<joint name="left_bump_mnt" type="fixed">
-		<origin xyz="-0.0256 0.0207 0.013" rpy="0 0 0"/>
-		<parent link="base_link"/>
-		<child link="left_bump"/>
-	</joint>
-	<joint name="right_bump_mnt" type="fixed">
-		<origin xyz="0.0256 0.0207 0.013" rpy="0 0 0"/>
-		<parent link="base_link"/>
-		<child link="right_bump"/>
-	</joint>
-	<joint name="left_front_bump_mnt" type="fixed">
-		<origin xyz="-0.009152 0.032074 0.013" rpy="0 0 0"/>
-		<parent link="base_link"/>
-		<child link="left_front_bump"/>
-	</joint>
-	<joint name="right_front_bump_mnt" type="fixed">
-		<origin xyz="0.009152 0.032074 0.013" rpy="0 0 0"/>
-		<parent link="base_link"/>
-		<child link="right_front_bump"/>
-	</joint>
-	<gazebo reference="left_bump_mnt">
-		<preserveFixedJoint>true</preserveFixedJoint>
-	</gazebo>
-	<gazebo reference="right_bump_mnt">
-		<preserveFixedJoint>true</preserveFixedJoint>
-	</gazebo>
-	<gazebo reference="left_front_bump_mnt">
-		<preserveFixedJoint>true</preserveFixedJoint>
-	</gazebo>
-	<gazebo reference="right_front_bump_mnt">
-		<preserveFixedJoint>true</preserveFixedJoint>
-	</gazebo>
-	<gazebo reference="left_bump">
-		<mu1>1.0</mu1>
-		<mu2>1.0</mu2>
-		<kp>1000000.0</kp>
-		<kd>100.0</kd>
-		<minDepth>0.001</minDepth>
-		<maxVel>1.0</maxVel>
-		<material>Gazebo/Blue</material>
-		<sensor name="left_bump" type="contact">
-			<updateRate>30</updateRate>
-			<contact>
-				<collision>left_bump_collision_collision</collision>
-			</contact>
-			<plugin name="gazebo_ros_bumper" filename="libgazebo_ros_bumper.so">
-				<bumperTopicName>bumper</bumperTopicName>
-				<frameName>left_bump</frameName>
-			</plugin>
-		</sensor>
-	</gazebo>
-	<gazebo reference="right_bump">
-		<mu1>1.0</mu1>
-		<mu2>1.0</mu2>
-		<kp>1000000.0</kp>
-		<kd>100.0</kd>
-		<minDepth>0.001</minDepth>
-		<maxVel>1.0</maxVel>
-		<material>Gazebo/Blue</material>
-		<sensor name="right_bump" type="contact">
-			<updateRate>30</updateRate>
-			<contact>
-				<collision>right_bump_collision_collision</collision>
-			</contact>
-			<plugin name="gazebo_ros_bumper" filename="libgazebo_ros_bumper.so">
-				<bumperTopicName>bumper</bumperTopicName>
-				<frameName>right_bump</frameName>
-			</plugin>
-		</sensor>
-	</gazebo>
-	<gazebo reference="left_front_bump">
-		<mu1>1.0</mu1>
-		<mu2>1.0</mu2>
-		<kp>1000000.0</kp>
-		<kd>100.0</kd>
-		<minDepth>0.001</minDepth>
-		<maxVel>1.0</maxVel>
-		<material>Gazebo/Blue</material>
-		<sensor name="left_front_bump" type="contact">
-			<updateRate>30</updateRate>
-			<contact>
-				<collision>left_front_bump_collision_collision</collision>
-			</contact>
-			<plugin name="gazebo_ros_bumper" filename="libgazebo_ros_bumper.so">
-				<bumperTopicName>bumper</bumperTopicName>
-				<frameName>left_front_bump</frameName>
-			</plugin>
-		</sensor>
-	</gazebo>
-	<gazebo reference="right_front_bump">
-		<mu1>1.0</mu1>
-		<mu2>1.0</mu2>
-		<kp>1000000.0</kp>
-		<kd>100.0</kd>
-		<minDepth>0.001</minDepth>
-		<maxVel>1.0</maxVel>
-		<material>Gazebo/Blue</material>
-		<sensor name="right_front_bump" type="contact">
-			<updateRate>30</updateRate>
-			<contact>
-				<collision>right_front_bump_collision_collision</collision>
-			</contact>
-			<plugin name="gazebo_ros_bumper" filename="libgazebo_ros_bumper.so">
-				<bumperTopicName>bumper</bumperTopicName>
-				<frameName>right_front_bump</frameName>
-			</plugin>
-		</sensor>
-	</gazebo>
-	<!-- TODO add compass sensor -->
-	<!-- TODO add GPS sensor -->
 </robot>
