Commit message: Added laser sensors

File: mouse_description/urdf/ant.xacro (robot description, xacro)
@@ -5,4 +5,5 @@
 	<xacro:property name="wheel_torque" value="0.015"/>
 	<xacro:property name="wheel_veloc" value="105"/>
+	<xacro:property name="ir_max" value="0.2"/>
 	<link name="base_link">
 		<visual>
@@ -15,9 +16,4 @@
 				<mesh filename="package://mouse_description/meshes/mouse_base.dae" scale="1 1 1"/>
 			</geometry>
-			<surface>
-				<contact>
-					<collide_bitmask>0x0</collide_bitmask>
-				</contact>
-			</surface>
 		</collision>
 		<inertial>
@@ -30,4 +26,59 @@
 		</inertial>
 	</link>
+	<!-- Actuation -->
+	<link name="left_wheel">
+		<visual>
+			<geometry>
+				<mesh filename="package://mouse_description/meshes/mouse_wheel.dae" scale="1 1 1"/>
+			</geometry>
+		</visual>
+		<collision name="left_wheel_collision">
+			<geometry>
+				<mesh filename="package://mouse_description/meshes/mouse_wheel.dae" scale="1 1 1"/>
+			</geometry>
+		</collision>
+		<inertial>
+			<mass value="0.015"/>
+			<inertia
+        		ixx="2.196e-6" ixy="0.0" ixz="0.0"
+        		iyy="1.146e-6" iyz="0.0"
+        		izz="1.146e-6"/>
+		</inertial>
+	</link>
+	<link name="right_wheel">
+		<visual>
+			<geometry>
+				<mesh filename="package://mouse_description/meshes/mouse_wheel.dae" scale="1 1 1"/>
+			</geometry>
+		</visual>
+		<collision name="right_wheel_collision">
+			<geometry>
+				<mesh filename="package://mouse_description/meshes/mouse_wheel.dae" scale="1 1 1"/>
+			</geometry>
+		</collision>
+		<inertial>
+			<mass value="0.015"/>
+			<inertia
+        		ixx="2.196e-6" ixy="0.0" ixz="0.0"
+        		iyy="1.146e-6" iyz="0.0"
+        		izz="1.146e-6"/>
+		</inertial>
+	</link>
+	<joint name="left_mot" type="continuous">
+		<parent link="base_link"/>
+		<child link="left_wheel"/>
+		<origin xyz="${wheel_sep/2} 0 ${wheel_dia/2}" rpy="0 0 0"/>
+		<axis xyz="-1 0 0"/>
+		<dynamics friction="0.01"/>
+		<limit effort="${wheel_torque}" velocity="${wheel_veloc}"/>
+	</joint>
+	<joint name="right_mot" type="continuous">
+		<parent link="base_link"/>
+		<child link="right_wheel"/>
+		<origin xyz="${-wheel_sep/2} 0 ${wheel_dia/2}" rpy="0 0 0"/>
+		<axis xyz="-1 0 0"/>
+		<dynamics friction="0.01"/>
+		<limit effort="${wheel_torque}" velocity="${wheel_veloc}"/>
+	</joint>
 	<gazebo reference="base_link">
 		<mu1>0.1</mu1>
@@ -39,72 +90,7 @@
 		<material>Gazebo/Blue</material>
 	</gazebo>
-	<!-- Actuation -->
-	<link name="left_wheel">
-		<visual>
-			<geometry>
-				<mesh filename="package://mouse_description/meshes/mouse_wheel.dae" scale="1 1 1"/>
-			</geometry>
-		</visual>
-		<collision name="left_wheel_collision">
-			<geometry>
-				<mesh filename="package://mouse_description/meshes/mouse_wheel.dae" scale="1 1 1"/>
-			</geometry>
-			<surface>
-				<contact>
-					<collide_bitmask>0x0</collide_bitmask>
-				</contact>
-			</surface>
-		</collision>
-		<inertial>
-			<mass value="0.015"/>
-			<inertia
-        		ixx="2.196e-6" ixy="0.0" ixz="0.0"
-        		iyy="1.146e-6" iyz="0.0"
-        		izz="1.146e-6"/>
-		</inertial>
-	</link>
-	<link name="right_wheel">
-		<visual>
-			<geometry>
-				<mesh filename="package://mouse_description/meshes/mouse_wheel.dae" scale="1 1 1"/>
-			</geometry>
-		</visual>
-		<collision name="right_wheel_collision">
-			<geometry>
-				<mesh filename="package://mouse_description/meshes/mouse_wheel.dae" scale="1 1 1"/>
-			</geometry>
-			<surface>
-				<contact>
-					<collide_bitmask>0x0</collide_bitmask>
-				</contact>
-			</surface>
-		</collision>
-		<inertial>
-			<mass value="0.015"/>
-			<inertia
-        		ixx="2.196e-6" ixy="0.0" ixz="0.0"
-        		iyy="1.146e-6" iyz="0.0"
-        		izz="1.146e-6"/>
-		</inertial>
-	</link>
-	<joint name="left_mot" type="continuous">
-		<parent link="base_link"/>
-		<child link="left_wheel"/>
-		<origin xyz="${wheel_sep/2} 0 ${wheel_dia/2}" rpy="0 0 0"/>
-		<axis xyz="-1 0 0"/>
-		<dynamics friction="0.001"/>
-		<limit effort="${wheel_torque}" velocity="${wheel_veloc}"/>
-	</joint>
-	<joint name="right_mot" type="continuous">
-		<parent link="base_link"/>
-		<child link="right_wheel"/>
-		<origin xyz="${-wheel_sep/2} 0 ${wheel_dia/2}" rpy="0 0 0"/>
-		<axis xyz="-1 0 0"/>
-		<dynamics friction="0.001"/>
-		<limit effort="${wheel_torque}" velocity="${wheel_veloc}"/>
-	</joint>
 	<gazebo reference="left_wheel">
-		<mu1>100.0</mu1>
-		<mu2>100.0</mu2>
+		<mu1>1000.0</mu1>
+		<mu2>1000.0</mu2>
 		<kp>1000000.0</kp>
 		<kd>100.0</kd>
@@ -114,6 +100,6 @@
 	</gazebo>
 	<gazebo reference="right_wheel">
-		<mu1>100.0</mu1>
-		<mu2>100.0</mu2>
+		<mu1>1000.0</mu1>
+		<mu2>1000.0</mu2>
 		<kp>1000000.0</kp>
 		<kd>100.0</kd>
@@ -146,3 +132,142 @@
 		</plugin>
 	</gazebo>
+	<!-- Sensors -->
+	<link name="left_ir">
+		<visual>
+			<geometry>
+				<sphere radius="0.001"/>
+			</geometry>
+		</visual>
+		<inertial>
+			<mass value="1e-5"/>
+			<inertia
+				ixx="1e-6" ixy="0.0" ixz="0.0"
+				iyy="1e-6" iyz="0.0"
+				izz="1e-6"/>
+		</inertial>
+	</link>
+	<joint name="left_ir_mnt" type="fixed">
+		<origin xyz="-0.0256 0.0207 0.020" rpy="0 0 3.14159265359"/>
+		<parent link="base_link"/>
+		<child link="left_ir"/>
+	</joint>
+	<gazebo reference="left_ir">
+		<material>Gazebo/Red</material>
+		<sensor type="ray" name="left_ir_sens">
+			<pose>0 0 0 0 0 0</pose>
+			<visualize>true</visualize>
+			<update_rate>30</update_rate>
+			<ray>
+				<scan>
+					<horizontal>
+						<samples>3</samples>
+						<resolution>1</resolution>
+						<min_angle>-0.03</min_angle>
+						<max_angle>0.03</max_angle>
+					</horizontal>
+				</scan>
+				<range>
+					<min>0.001</min>
+					<max>${ir_max}</max>
+					<resolution>0.001</resolution>
+				</range>
+			</ray>
+			<plugin filename="libgazebo_ros_laser.so" name="gazebo_ros_laser">
+				<topicName>laser</topicName>
+				<frameName>left_ir</frameName>
+			</plugin>
+		</sensor>
+	</gazebo>
+	<link name="right_ir">
+		<visual>
+			<geometry>
+				<sphere radius="0.001"/>
+			</geometry>
+		</visual>
+		<inertial>
+			<mass value="1e-5"/>
+			<inertia
+				ixx="1e-6" ixy="0.0" ixz="0.0"
+				iyy="1e-6" iyz="0.0"
+				izz="1e-6"/>
+		</inertial>
+	</link>
+	<joint name="right_ir_mnt" type="fixed">
+		<origin xyz="0.0256 0.0207 0.020" rpy="0 0 0"/>
+		<parent link="base_link"/>
+		<child link="right_ir"/>
+	</joint>
+	<gazebo reference="right_ir">
+		<material>Gazebo/Red</material>
+		<sensor type="ray" name="right_ir_sens">
+			<pose>0 0 0 0 0 0</pose>
+			<visualize>true</visualize>
+			<update_rate>30</update_rate>
+			<ray>
+				<scan>
+					<horizontal>
+						<samples>3</samples>
+						<resolution>1</resolution>
+						<min_angle>-0.03</min_angle>
+						<max_angle>0.03</max_angle>
+					</horizontal>
+				</scan>
+				<range>
+					<min>0.001</min>
+					<max>${ir_max}</max>
+					<resolution>0.001</resolution>
+				</range>
+			</ray>
+			<plugin filename="libgazebo_ros_laser.so" name="gazebo_ros_laser">
+				<topicName>laser</topicName>
+				<frameName>right_ir</frameName>
+			</plugin>
+		</sensor>
+	</gazebo>
+	<link name="center_ir">
+		<visual>
+			<geometry>
+				<sphere radius="0.001"/>
+			</geometry>
+		</visual>
+		<inertial>
+			<mass value="1e-5"/>
+			<inertia
+				ixx="1e-6" ixy="0.0" ixz="0.0"
+				iyy="1e-6" iyz="0.0"
+				izz="1e-6"/>
+		</inertial>
+	</link>
+	<joint name="center_ir_mnt" type="fixed">
+		<origin xyz="0 0.03 0.020" rpy="0 0 1.57079632679"/>
+		<parent link="base_link"/>
+		<child link="center_ir"/>
+	</joint>
+	<gazebo reference="center_ir">
+		<material>Gazebo/Red</material>
+		<sensor type="ray" name="center_ir_sens">
+			<pose>0 0 0 0 0 0</pose>
+			<visualize>true</visualize>
+			<update_rate>30</update_rate>
+			<ray>
+				<scan>
+					<horizontal>
+						<samples>3</samples>
+						<resolution>1</resolution>
+						<min_angle>-0.03</min_angle>
+						<max_angle>0.03</max_angle>
+					</horizontal>
+				</scan>
+				<range>
+					<min>0.001</min>
+					<max>${ir_max}</max>
+					<resolution>0.001</resolution>
+				</range>
+			</ray>
+			<plugin filename="libgazebo_ros_laser.so" name="gazebo_ros_laser">
+				<topicName>laser</topicName>
+				<frameName>center_ir</frameName>
+			</plugin>
+		</sensor>
+	</gazebo>
 </robot>

File: mouse_description/urdf/bee.xacro (robot description, xacro)
@@ -5,4 +5,5 @@
 	<xacro:property name="wheel_torque" value="0.015"/>
 	<xacro:property name="wheel_veloc" value="105"/>
+	<xacro:property name="ir_max" value="0.2"/>
 	<link name="base_link">
 		<visual>
@@ -15,9 +16,4 @@
 				<mesh filename="package://mouse_description/meshes/mouse_base.dae" scale="1 1 1"/>
 			</geometry>
-			<surface>
-				<contact>
-					<collide_bitmask>0x0</collide_bitmask>
-				</contact>
-			</surface>
 		</collision>
 		<inertial>
@@ -30,4 +26,59 @@
 		</inertial>
 	</link>
+	<!-- Actuation -->
+	<link name="left_wheel">
+		<visual>
+			<geometry>
+				<mesh filename="package://mouse_description/meshes/mouse_wheel.dae" scale="1 1 1"/>
+			</geometry>
+		</visual>
+		<collision name="left_wheel_collision">
+			<geometry>
+				<mesh filename="package://mouse_description/meshes/mouse_wheel.dae" scale="1 1 1"/>
+			</geometry>
+		</collision>
+		<inertial>
+			<mass value="0.015"/>
+			<inertia
+        		ixx="2.196e-6" ixy="0.0" ixz="0.0"
+        		iyy="1.146e-6" iyz="0.0"
+        		izz="1.146e-6"/>
+		</inertial>
+	</link>
+	<link name="right_wheel">
+		<visual>
+			<geometry>
+				<mesh filename="package://mouse_description/meshes/mouse_wheel.dae" scale="1 1 1"/>
+			</geometry>
+		</visual>
+		<collision name="right_wheel_collision">
+			<geometry>
+				<mesh filename="package://mouse_description/meshes/mouse_wheel.dae" scale="1 1 1"/>
+			</geometry>
+		</collision>
+		<inertial>
+			<mass value="0.015"/>
+			<inertia
+        		ixx="2.196e-6" ixy="0.0" ixz="0.0"
+        		iyy="1.146e-6" iyz="0.0"
+        		izz="1.146e-6"/>
+		</inertial>
+	</link>
+	<joint name="left_mot" type="continuous">
+		<parent link="base_link"/>
+		<child link="left_wheel"/>
+		<origin xyz="${wheel_sep/2} 0 ${wheel_dia/2}" rpy="0 0 0"/>
+		<axis xyz="-1 0 0"/>
+		<dynamics friction="0.01"/>
+		<limit effort="${wheel_torque}" velocity="${wheel_veloc}"/>
+	</joint>
+	<joint name="right_mot" type="continuous">
+		<parent link="base_link"/>
+		<child link="right_wheel"/>
+		<origin xyz="${-wheel_sep/2} 0 ${wheel_dia/2}" rpy="0 0 0"/>
+		<axis xyz="-1 0 0"/>
+		<dynamics friction="0.01"/>
+		<limit effort="${wheel_torque}" velocity="${wheel_veloc}"/>
+	</joint>
 	<gazebo reference="base_link">
 		<mu1>0.1</mu1>
@@ -39,72 +90,7 @@
 		<material>Gazebo/Yellow</material>
 	</gazebo>
-	<!-- Actuation -->
-	<link name="left_wheel">
-		<visual>
-			<geometry>
-				<mesh filename="package://mouse_description/meshes/mouse_wheel.dae" scale="1 1 1"/>
-			</geometry>
-		</visual>
-		<collision name="left_wheel_collision">
-			<geometry>
-				<mesh filename="package://mouse_description/meshes/mouse_wheel.dae" scale="1 1 1"/>
-			</geometry>
-			<surface>
-				<contact>
-					<collide_bitmask>0x0</collide_bitmask>
-				</contact>
-			</surface>
-		</collision>
-		<inertial>
-			<mass value="0.015"/>
-			<inertia
-        		ixx="2.196e-6" ixy="0.0" ixz="0.0"
-        		iyy="1.146e-6" iyz="0.0"
-        		izz="1.146e-6"/>
-		</inertial>
-	</link>
-	<link name="right_wheel">
-		<visual>
-			<geometry>
-				<mesh filename="package://mouse_description/meshes/mouse_wheel.dae" scale="1 1 1"/>
-			</geometry>
-		</visual>
-		<collision name="right_wheel_collision">
-			<geometry>
-				<mesh filename="package://mouse_description/meshes/mouse_wheel.dae" scale="1 1 1"/>
-			</geometry>
-			<surface>
-				<contact>
-					<collide_bitmask>0x0</collide_bitmask>
-				</contact>
-			</surface>
-		</collision>
-		<inertial>
-			<mass value="0.015"/>
-			<inertia
-        		ixx="2.196e-6" ixy="0.0" ixz="0.0"
-        		iyy="1.146e-6" iyz="0.0"
-        		izz="1.146e-6"/>
-		</inertial>
-	</link>
-	<joint name="left_mot" type="continuous">
-		<parent link="base_link"/>
-		<child link="left_wheel"/>
-		<origin xyz="${wheel_sep/2} 0 ${wheel_dia/2}" rpy="0 0 0"/>
-		<axis xyz="-1 0 0"/>
-		<dynamics friction="0.001"/>
-		<limit effort="${wheel_torque}" velocity="${wheel_veloc}"/>
-	</joint>
-	<joint name="right_mot" type="continuous">
-		<parent link="base_link"/>
-		<child link="right_wheel"/>
-		<origin xyz="${-wheel_sep/2} 0 ${wheel_dia/2}" rpy="0 0 0"/>
-		<axis xyz="-1 0 0"/>
-		<dynamics friction="0.001"/>
-		<limit effort="${wheel_torque}" velocity="${wheel_veloc}"/>
-	</joint>
 	<gazebo reference="left_wheel">
-		<mu1>100.0</mu1>
-		<mu2>100.0</mu2>
+		<mu1>1000.0</mu1>
+		<mu2>1000.0</mu2>
 		<kp>1000000.0</kp>
 		<kd>100.0</kd>
@@ -114,6 +100,6 @@
 	</gazebo>
 	<gazebo reference="right_wheel">
-		<mu1>100.0</mu1>
-		<mu2>100.0</mu2>
+		<mu1>1000.0</mu1>
+		<mu2>1000.0</mu2>
 		<kp>1000000.0</kp>
 		<kd>100.0</kd>
@@ -146,3 +132,142 @@
 		</plugin>
 	</gazebo>
+	<!-- Sensors -->
+	<link name="left_ir">
+		<visual>
+			<geometry>
+				<sphere radius="0.001"/>
+			</geometry>
+		</visual>
+		<inertial>
+			<mass value="1e-5"/>
+			<inertia
+				ixx="1e-6" ixy="0.0" ixz="0.0"
+				iyy="1e-6" iyz="0.0"
+				izz="1e-6"/>
+		</inertial>
+	</link>
+	<joint name="left_ir_mnt" type="fixed">
+		<origin xyz="-0.0256 0.0207 0.020" rpy="0 0 3.14159265359"/>
+		<parent link="base_link"/>
+		<child link="left_ir"/>
+	</joint>
+	<gazebo reference="left_ir">
+		<material>Gazebo/Red</material>
+		<sensor type="ray" name="left_ir_sens">
+			<pose>0 0 0 0 0 0</pose>
+			<visualize>true</visualize>
+			<update_rate>30</update_rate>
+			<ray>
+				<scan>
+					<horizontal>
+						<samples>3</samples>
+						<resolution>1</resolution>
+						<min_angle>-0.03</min_angle>
+						<max_angle>0.03</max_angle>
+					</horizontal>
+				</scan>
+				<range>
+					<min>0.001</min>
+					<max>${ir_max}</max>
+					<resolution>0.001</resolution>
+				</range>
+			</ray>
+			<plugin filename="libgazebo_ros_laser.so" name="gazebo_ros_laser">
+				<topicName>laser</topicName>
+				<frameName>left_ir</frameName>
+			</plugin>
+		</sensor>
+	</gazebo>
+	<link name="right_ir">
+		<visual>
+			<geometry>
+				<sphere radius="0.001"/>
+			</geometry>
+		</visual>
+		<inertial>
+			<mass value="1e-5"/>
+			<inertia
+				ixx="1e-6" ixy="0.0" ixz="0.0"
+				iyy="1e-6" iyz="0.0"
+				izz="1e-6"/>
+		</inertial>
+	</link>
+	<joint name="right_ir_mnt" type="fixed">
+		<origin xyz="0.0256 0.0207 0.020" rpy="0 0 0"/>
+		<parent link="base_link"/>
+		<child link="right_ir"/>
+	</joint>
+	<gazebo reference="right_ir">
+		<material>Gazebo/Red</material>
+		<sensor type="ray" name="right_ir_sens">
+			<pose>0 0 0 0 0 0</pose>
+			<visualize>true</visualize>
+			<update_rate>30</update_rate>
+			<ray>
+				<scan>
+					<horizontal>
+						<samples>3</samples>
+						<resolution>1</resolution>
+						<min_angle>-0.03</min_angle>
+						<max_angle>0.03</max_angle>
+					</horizontal>
+				</scan>
+				<range>
+					<min>0.001</min>
+					<max>${ir_max}</max>
+					<resolution>0.001</resolution>
+				</range>
+			</ray>
+			<plugin filename="libgazebo_ros_laser.so" name="gazebo_ros_laser">
+				<topicName>laser</topicName>
+				<frameName>right_ir</frameName>
+			</plugin>
+		</sensor>
+	</gazebo>
+	<link name="center_ir">
+		<visual>
+			<geometry>
+				<sphere radius="0.001"/>
+			</geometry>
+		</visual>
+		<inertial>
+			<mass value="1e-5"/>
+			<inertia
+				ixx="1e-6" ixy="0.0" ixz="0.0"
+				iyy="1e-6" iyz="0.0"
+				izz="1e-6"/>
+		</inertial>
+	</link>
+	<joint name="center_ir_mnt" type="fixed">
+		<origin xyz="0 0.03 0.020" rpy="0 0 1.57079632679"/>
+		<parent link="base_link"/>
+		<child link="center_ir"/>
+	</joint>
+	<gazebo reference="center_ir">
+		<material>Gazebo/Red</material>
+		<sensor type="ray" name="center_ir_sens">
+			<pose>0 0 0 0 0 0</pose>
+			<visualize>true</visualize>
+			<update_rate>30</update_rate>
+			<ray>
+				<scan>
+					<horizontal>
+						<samples>3</samples>
+						<resolution>1</resolution>
+						<min_angle>-0.03</min_angle>
+						<max_angle>0.03</max_angle>
+					</horizontal>
+				</scan>
+				<range>
+					<min>0.001</min>
+					<max>${ir_max}</max>
+					<resolution>0.001</resolution>
+				</range>
+			</ray>
+			<plugin filename="libgazebo_ros_laser.so" name="gazebo_ros_laser">
+				<topicName>laser</topicName>
+				<frameName>center_ir</frameName>
+			</plugin>
+		</sensor>
+	</gazebo>
 </robot>

File: mouse_description/urdf/mouse.xacro (robot description, xacro)
@@ -5,4 +5,5 @@
 	<xacro:property name="wheel_torque" value="0.015"/>
 	<xacro:property name="wheel_veloc" value="105"/>
+	<xacro:property name="ir_max" value="0.2"/>
 	<link name="base_link">
 		<visual>
@@ -89,6 +90,6 @@
 	</joint>
 	<gazebo reference="left_wheel">
-		<mu1>1.0</mu1>
-		<mu2>1.0</mu2>
+		<mu1>1000.0</mu1>
+		<mu2>1000.0</mu2>
 		<kp>1000000.0</kp>
 		<kd>100.0</kd>
@@ -98,6 +99,6 @@
 	</gazebo>
 	<gazebo reference="right_wheel">
-		<mu1>1.0</mu1>
-		<mu2>1.0</mu2>
+		<mu1>1000.0</mu1>
+		<mu2>1000.0</mu2>
 		<kp>1000000.0</kp>
 		<kd>100.0</kd>
@@ -130,3 +131,142 @@
 		</plugin>
 	</gazebo>
+	<!-- Sensors -->
+	<link name="left_ir">
+		<visual>
+			<geometry>
+				<sphere radius="0.001"/>
+			</geometry>
+		</visual>
+		<inertial>
+			<mass value="1e-5"/>
+			<inertia
+				ixx="1e-6" ixy="0.0" ixz="0.0"
+				iyy="1e-6" iyz="0.0"
+				izz="1e-6"/>
+		</inertial>
+	</link>
+	<joint name="left_ir_mnt" type="fixed">
+		<origin xyz="-0.0256 0.0207 0.020" rpy="0 0 3.14159265359"/>
+		<parent link="base_link"/>
+		<child link="left_ir"/>
+	</joint>
+	<gazebo reference="left_ir">
+		<material>Gazebo/Red</material>
+		<sensor type="ray" name="left_ir_sens">
+			<pose>0 0 0 0 0 0</pose>
+			<visualize>true</visualize>
+			<update_rate>30</update_rate>
+			<ray>
+				<scan>
+					<horizontal>
+						<samples>3</samples>
+						<resolution>1</resolution>
+						<min_angle>-0.03</min_angle>
+						<max_angle>0.03</max_angle>
+					</horizontal>
+				</scan>
+				<range>
+					<min>0.001</min>
+					<max>${ir_max}</max>
+					<resolution>0.001</resolution>
+				</range>
+			</ray>
+			<plugin filename="libgazebo_ros_laser.so" name="gazebo_ros_laser">
+				<topicName>laser</topicName>
+				<frameName>left_ir</frameName>
+			</plugin>
+		</sensor>
+	</gazebo>
+	<link name="right_ir">
+		<visual>
+			<geometry>
+				<sphere radius="0.001"/>
+			</geometry>
+		</visual>
+		<inertial>
+			<mass value="1e-5"/>
+			<inertia
+				ixx="1e-6" ixy="0.0" ixz="0.0"
+				iyy="1e-6" iyz="0.0"
+				izz="1e-6"/>
+		</inertial>
+	</link>
+	<joint name="right_ir_mnt" type="fixed">
+		<origin xyz="0.0256 0.0207 0.020" rpy="0 0 0"/>
+		<parent link="base_link"/>
+		<child link="right_ir"/>
+	</joint>
+	<gazebo reference="right_ir">
+		<material>Gazebo/Red</material>
+		<sensor type="ray" name="right_ir_sens">
+			<pose>0 0 0 0 0 0</pose>
+			<visualize>true</visualize>
+			<update_rate>30</update_rate>
+			<ray>
+				<scan>
+					<horizontal>
+						<samples>3</samples>
+						<resolution>1</resolution>
+						<min_angle>-0.03</min_angle>
+						<max_angle>0.03</max_angle>
+					</horizontal>
+				</scan>
+				<range>
+					<min>0.001</min>
+					<max>${ir_max}</max>
+					<resolution>0.001</resolution>
+				</range>
+			</ray>
+			<plugin filename="libgazebo_ros_laser.so" name="gazebo_ros_laser">
+				<topicName>laser</topicName>
+				<frameName>right_ir</frameName>
+			</plugin>
+		</sensor>
+	</gazebo>
+	<link name="center_ir">
+		<visual>
+			<geometry>
+				<sphere radius="0.001"/>
+			</geometry>
+		</visual>
+		<inertial>
+			<mass value="1e-5"/>
+			<inertia
+				ixx="1e-6" ixy="0.0" ixz="0.0"
+				iyy="1e-6" iyz="0.0"
+				izz="1e-6"/>
+		</inertial>
+	</link>
+	<joint name="center_ir_mnt" type="fixed">
+		<origin xyz="0 0.03 0.020" rpy="0 0 1.57079632679"/>
+		<parent link="base_link"/>
+		<child link="center_ir"/>
+	</joint>
+	<gazebo reference="center_ir">
+		<material>Gazebo/Red</material>
+		<sensor type="ray" name="center_ir_sens">
+			<pose>0 0 0 0 0 0</pose>
+			<visualize>true</visualize>
+			<update_rate>30</update_rate>
+			<ray>
+				<scan>
+					<horizontal>
+						<samples>3</samples>
+						<resolution>1</resolution>
+						<min_angle>-0.03</min_angle>
+						<max_angle>0.03</max_angle>
+					</horizontal>
+				</scan>
+				<range>
+					<min>0.001</min>
+					<max>${ir_max}</max>
+					<resolution>0.001</resolution>
+				</range>
+			</ray>
+			<plugin filename="libgazebo_ros_laser.so" name="gazebo_ros_laser">
+				<topicName>laser</topicName>
+				<frameName>center_ir</frameName>
+			</plugin>
+		</sensor>
+	</gazebo>
 </robot>
