Commit message: Added map parsing

File: mouse_gazebo/models/box.xacro (robot description, xacro)
@@ -1,7 +1,6 @@
 <?xml version="1.0" ?>
 <robot name="box" xmlns:xacro="http://www.ros.org/wiki/xacro">
-<!-- TODO adjust parameters -->
-	<xacro:property name="len" value="0.25"/>
-	<xacro:property name="mass" value="0.5"/>
+	<xacro:property name="len" value="0.099"/>
+	<xacro:property name="mass" value="1"/>
 	<link name="base_link">
 		<visual>
@@ -26,9 +25,8 @@
 		</inertial>
 	</link>
-<!-- TODO change friction -->
 	<gazebo reference="base_link">
-		<mu1>0.1</mu1>
-		<mu2>0.1</mu2>
-		<material>Gazebo/Blue</material>
+		<mu1>1000000.0</mu1>
+		<mu2>1000000.0</mu2>
+		<material>Gazebo/Black</material>
 	</gazebo>
 </robot>

Commit message: Increased grid size

File: mouse_gazebo/models/box.xacro (robot description, xacro)
@@ -1,26 +1,26 @@
 <?xml version="1.0" ?>
 <robot name="box" xmlns:xacro="http://www.ros.org/wiki/xacro">
-	<xacro:property name="len" value="0.099"/>
+	<xacro:property name="grid_size" value="0.179"/>
 	<xacro:property name="mass" value="1"/>
 	<link name="base_link">
 		<visual>
-			<origin xyz="0 0 ${len/2}" rpy="0 0 0"/>
+			<origin xyz="0 0 ${grid_size/2}" rpy="0 0 0"/>
 			<geometry>
-				<box size="${len} ${len} ${len}"/>
+				<box size="${grid_size} ${grid_size} ${grid_size}"/>
 			</geometry>
 		</visual>
 		<collision>
-			<origin xyz="0 0 ${len/2}" rpy="0 0 0"/>
+			<origin xyz="0 0 ${grid_size/2}" rpy="0 0 0"/>
 			<geometry>
-				<box size="${len} ${len} ${len}"/>
+				<box size="${grid_size} ${grid_size} ${grid_size}"/>
 			</geometry>
 		</collision>
 		<inertial>
-			<origin xyz="0 0 ${len/2}" rpy="0 0 0"/>
+			<origin xyz="0 0 ${grid_size/2}" rpy="0 0 0"/>
 			<mass value="${mass}"/>
 			<inertia
-        		ixx="${1/6*mass*len*len}" ixy="0.0" ixz="0.0"
-        		iyy="${1/6*mass*len*len}" iyz="0.0"
-        		izz="${1/6*mass*len*len}"/>
+        		ixx="${1/6*mass*grid_size*grid_size}" ixy="0.0" ixz="0.0"
+        		iyy="${1/6*mass*grid_size*grid_size}" iyz="0.0"
+        		izz="${1/6*mass*grid_size*grid_size}"/>
 		</inertial>
 	</link>

File: mouse_gazebo/models/divider.xacro (robot description, xacro)
@@ -1,9 +1,10 @@
 <?xml version="1.0" ?>
 <robot name="box" xmlns:xacro="http://www.ros.org/wiki/xacro">
+	<xacro:property name="grid_size" value="0.180"/>
 	<link name="base_link">
 		<visual>
 			<origin xyz="0 0 0.001" rpy="0 0 0"/>
 			<geometry>
-				<box size="0.1 0.004 0.002"/>
+				<box size="${grid_size} 0.004 0.002"/>
 			</geometry>
 		</visual>
